File: voltage-convertor-board/voltage-convertor-board.kicad_pcb (KiCad board)
At the start: 2 copper layers, 60 parts, among them IC1 MCP2562, J1 Conn_01x04, J10 Conn_01x02, J11 Conn_01x02, J2 Conn_01x03, J3 Conn_01x03, J4 Conn_01x04, J5 Conn_01x04, J6 Conn_01x04_Pin, J7 Conn_01x04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

Commit message: PCB　シルク、ビア、LED以外完成
Parts:
- added D2: LED, LED_SMD:LED_0603_1608Metric_Pad1.05x0.95mm_HandSolder, F.Cu at (18.0, 72.2)
- added D3: LED, LED_SMD:LED_0603_1608Metric_Pad1.05x0.95mm_HandSolder, F.Cu at (18.0, 73.8)
- added D4: LED, LED_SMD:LED_0603_1608Metric_Pad1.05x0.95mm_HandSolder, F.Cu at (18.0, 75.4)
- added R17: 1k, Resistor_SMD:R_0603_1608Metric_Pad0.98x0.95mm_HandSolder, F.Cu at (21.4, 72.2)
- added R18: 1k, Resistor_SMD:R_0603_1608Metric_Pad0.98x0.95mm_HandSolder, F.Cu at (21.4, 73.8)
- added R19: 1k, Resistor_SMD:R_0603_1608Metric_Pad0.98x0.95mm_HandSolder, F.Cu at (21.4, 75.4)
- added REF**: MountingHole_3.2mm_M3, MountingHole:MountingHole_3.2mm_M3, F.Cu at (19.0, 19.0)
- added REF**: MountingHole_3.2mm_M3, MountingHole:MountingHole_3.2mm_M3, F.Cu at (19.0, 81.0)
- added REF**: MountingHole_3.2mm_M3, MountingHole:MountingHole_3.2mm_M3, F.Cu at (71.0, 81.0)
- added REF**: MountingHole_3.2mm_M3, MountingHole:MountingHole_3.2mm_M3, F.Cu at (71.0, 19.0)
- C10, C12, C13, C9: footprint Capacitor_SMD:C_0603_1608Metric_Pad1.08x0.95mm_HandSolder -> Capacitor_SMD:C_1210_3225Metric_Pad1.33x2.70mm_HandSolder
- C14, J4, J5: moved to B.Cu
- J1: footprint Connector_JST:JST_XH_B4B-XH-A_1x04_P2.50mm_Vertical -> Connector_JST:JST_XH_S4B-XH-A_1x04_P2.50mm_Horizontal
- moved J6 60.3 mm to (25.0, 81.5), turned to 180 degrees
- moved F1 59.9 mm to (70.6, 25.6)
- moved U5 56.6 mm to (33.7, 64.2)
- moved J2 56.2 mm to (65.4, 69.0), turned to 90 degrees
- moved J11 51.7 mm to (62.4, 22.6)
- moved J1 47.7 mm to (24.9, 48.2), turned to -90 degrees
- moved D1 44.4 mm to (46.8, 37.2), turned to 180 degrees
- moved U1 43.0 mm to (45.8, 41.6)
- moved J10 41.2 mm to (27.4, 31.8)
- moved J5 41.1 mm to (63.8, 74.4), turned to 180 degrees
- moved J4 40.6 mm to (50.1, 74.7), turned to 180 degrees
- moved J3 40.1 mm to (65.4, 58.0), turned to 90 degrees
- moved SW1 36.5 mm to (17.0, 69.6)
- moved C19 35.6 mm to (32.4, 39.6), turned to 180 degrees
- moved R12 35.6 mm to (69.1, 73.3), turned to 180 degrees
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Connections:
- C19 pad 2: GND -> GNDD
- C6 pad 1: +5P -> +5VP
- J10 pad 1: GND -> GNDD
- J11 pad 1: GND -> GNDD
- JP1 pad 1: Net-(JP1-A) -> CANH
- JP1 pad 2: CANL -> Net-(JP1-B)
- Q2 pad 3: IN2 -> IN4
- R11 pad 2: IN2 -> IN4
- R12 pad 1: CANH -> Net-(JP1-B)
- R12 pad 2: Net-(JP1-A) -> CANL
- U5 pad 10: unconnected-(U5-PA5-Pad10) -> IN2
- U5 pad 11: unconnected-(U5-PA6-Pad11) -> IN3
- U5 pad 13: DIP2 -> unconnected-(U5-PB0-Pad13)
- U5 pad 26: TIM3_CH2 -> unconnected-(U5-PB3-Pad26)
- U5 pad 27: TIM3_CH1 -> unconnected-(U5-PB4-Pad27)
- U5 pad 28: DIP4 -> unconnected-(U5-PB5-Pad28)
- U5 pad 5: IN1 -> LED1
- U5 pad 6: IN2 -> LED2
- U5 pad 7: unconnected-(U5-PA2-Pad7) -> LED3
- U5 pad 8: unconnected-(U5-PA3-Pad8) -> IN4
- U5 pad 9: unconnected-(U5-PA4-Pad9) -> IN1
- U6 pad 3: +5P -> +5VP
Routing:
- net +3.3V: track 0.00 -> 94.0 mm, vias 0 -> 2
- net +12VA: track 0.00 -> 77.4 mm
- net +5V: track 0.00 -> 47.7 mm, vias 0 -> 3
- net CANH: track 0.00 -> 45.4 mm, vias 0 -> 1
- net Net-(J9-Pin_2): track 0.00 -> 40.6 mm, vias 0 -> 1
- net IN3: track 0.00 -> 33.7 mm, vias 0 -> 3
- net IN2: track 0.00 -> 32.4 mm, vias 0 -> 3
- net IN4: track 0.00 -> 32.4 mm, vias 0 -> 3
- net IN1: track 0.00 -> 31.7 mm, vias 0 -> 3
- net +12V: track 0.00 -> 31.0 mm
- net CANL: track 0.00 -> 30.8 mm, vias 0 -> 1
- net SWDIO: track 0.00 -> 28.9 mm, vias 0 -> 1
- net Net-(J8-Pin_2): track 0.00 -> 26.2 mm, vias 0 -> 1
- net SWCLK: track 0.00 -> 24.5 mm, vias 0 -> 1
- net UART_TX: track 0.00 -> 15.5 mm, vias 0 -> 1
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- added copper zone on B.Cu, net +12V
- added copper zone on F.Cu, net +12V
- added copper zone on B.Cu, net GNDD
- added copper zone on F.Cu, net GNDD
- added copper zone on F.Cu, net Net-(D1-K)
- added copper zone on B.Cu, net VCC
- added copper zone on F.Cu, net VCC
Other:
- board outline added: 60 x 70 mm
- board text added: "1 2 3"

Commit message: ビア以外完成
Parts:
- added D10: LED, LED_SMD:LED_0603_1608Metric_Pad1.05x0.95mm_HandSolder, F.Cu at (57.4, 81.5)
- added D5: LED, LED_SMD:LED_0603_1608Metric_Pad1.05x0.95mm_HandSolder, F.Cu at (46.4, 18.6)
- added D6: LED, LED_SMD:LED_0603_1608Metric_Pad1.05x0.95mm_HandSolder, F.Cu at (44.8, 18.6)
- added D7: LED, LED_SMD:LED_0603_1608Metric_Pad1.05x0.95mm_HandSolder, F.Cu at (43.2, 18.6)
- added D8: LED, LED_SMD:LED_0603_1608Metric_Pad1.05x0.95mm_HandSolder, F.Cu at (18.0, 76.4)
- added D9: LED, LED_SMD:LED_0603_1608Metric_Pad1.05x0.95mm_HandSolder, F.Cu at (59.0, 81.5)
- added R20: 1k, Resistor_SMD:R_0603_1608Metric_Pad0.98x0.95mm_HandSolder, F.Cu at (46.4, 22.0)
- added R21: 1k, Resistor_SMD:R_0603_1608Metric_Pad0.98x0.95mm_HandSolder, F.Cu at (44.8, 22.0)
- added R22: 1k, Resistor_SMD:R_0603_1608Metric_Pad0.98x0.95mm_HandSolder, F.Cu at (43.2, 22.0)
- added R23: 1k, Resistor_SMD:R_0603_1608Metric_Pad0.98x0.95mm_HandSolder, F.Cu at (21.4, 76.4)
- added R24: 1k, Resistor_SMD:R_0603_1608Metric_Pad0.98x0.95mm_HandSolder, F.Cu at (59.0, 78.1)
- added R25: 1k, Resistor_SMD:R_0603_1608Metric_Pad0.98x0.95mm_HandSolder, F.Cu at (57.4, 78.1)
- moved C14 1.93 mm to (58.8, 30.4), turned to 90 degrees
- moved D2 0.60 mm to (18.0, 71.6)
- moved D4 0.60 mm to (18.0, 74.8)
- moved R17 0.60 mm to (21.4, 71.6)
- moved R19 0.60 mm to (21.4, 74.8)
- moved D3 0.60 mm to (18.0, 73.2)
- moved R18 0.60 mm to (21.4, 73.2)
- moved SW1 0.20 mm to (17.2, 69.6)
Connections:
- U5 pad 10: IN2 -> IN1
- U5 pad 11: IN3 -> IN2
- U5 pad 12: unconnected-(U5-PA7-Pad12) -> IN3
- U5 pad 8: IN4 -> LED4
- U5 pad 9: IN1 -> IN4
Routing:
- net +5VP: track 8.45 -> 62.0 mm, vias 0 -> 1
- net VCC: track 14.7 -> 34.9 mm
- net +3.3V: track 94.0 -> 108.7 mm, vias 2 -> 4
- net LED4: track 0.00 -> 13.6 mm, vias 0 -> 2
- net +12V: track 31.0 -> 42.4 mm
- net +5V: track 47.7 -> 50.5 mm
- net Net-(D8-A): track 0.00 -> 1.61 mm
- net Net-(D9-A): track 0.00 -> 1.61 mm
- net Net-(D7-A): track 0.00 -> 1.61 mm
- net Net-(D6-A): track 0.00 -> 1.61 mm
- net Net-(D5-A): track 0.00 -> 1.61 mm
- net Net-(D10-A): track 0.00 -> 1.61 mm
- net IN3: track 33.7 -> 33.1 mm
- net LED1: track 11.7 -> 11.1 mm
- net LED3: track 13.5 -> 12.9 mm
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Other:
- board text added: "1 2 3 4"
- board text added: "12"
- board text added: "3.3 5"
- board text added: "5"
- board text added: "VCC"
- board text removed: "1 2 3"

Commit message: 完成
Parts:
- added D11: LED, LED_SMD:LED_0603_1608Metric_Pad1.05x0.95mm_HandSolder, F.Cu at (46.4, 18.6)
- added G***: LOGO, LOGO, F.Cu at (17.8, 41.2)
- added R26: 1k, Resistor_SMD:R_0603_1608Metric_Pad0.98x0.95mm_HandSolder, F.Cu at (46.4, 22.0)
- moved D5 1.60 mm to (48.0, 18.6)
- moved R20 1.60 mm to (48.0, 22.0)
Routing:
- net +12VA: track 77.4 -> 109.3 mm, vias 0 -> 2
- net Net-(D11-A): track 0.00 -> 1.61 mm
- net VCC: track 34.9 -> 36.5 mm, vias 4 -> 16
- net +12V: track 42.4 -> 42.7 mm, vias 0 -> 24
- net GNDD: vias 2 -> 210
Other:
- board text added: "1"
- board text added: "2"
- board text added: "5V出力"
- board text added: "CAN"
- board text added: "F"
- board text added: "G NC 5 NC"
- board text added: "H 5 L G"
- board text added: "R 3.3 T G"
- board text added: "UART"
- board text added: "voltage-convertor-board version 1.0 create by ikeda"
