File: voltage-convertor-board/voltage-convertor-board.kicad_sch (KiCad schematic)
At the start: 60 parts, among them IC1 MCP2562, J1 Conn_01x04, J10 Conn_01x02, J11 Conn_01x02, J2 Conn_01x03, J3 Conn_01x03, J4 Conn_01x04, J5 Conn_01x04, J6 Conn_01x04_Pin, J7 Conn_01x04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

Commit message: PCB　シルク、ビア、LED以外完成
Parts:
- added D2, D3, D4: LED, LED_SMD:LED_0603_1608Metric_Pad1.05x0.95mm_HandSolder, symbol Device:LED
- added R17, R18, R19: 1k, Resistor_SMD:R_0603_1608Metric_Pad0.98x0.95mm_HandSolder, symbol Device:R
- C10, C12, C13, C9: footprint Capacitor_SMD:C_0603_1608Metric_Pad1.08x0.95mm_HandSolder -> Capacitor_SMD:C_1210_3225Metric_Pad1.33x2.70mm_HandSolder
- J1: footprint Connector_JST:JST_XH_B4B-XH-A_1x04_P2.50mm_Vertical -> Connector_JST:JST_XH_S4B-XH-A_1x04_P2.50mm_Horizontal
Connections:
- net +5P is gone; now on net +5VP: C6.1, U6.3 (VOUT)
- net GND is gone; now on net GNDD: C19.2, J10.1 (Pin_1), J11.1 (Pin_1)
- net CANH: now also JP1.1 (A); no longer R12.1
- net CANL: now also R12.2; no longer JP1.2 (B)
- net GNDD: now also D2.1 (K), D3.1 (K), D4.1 (K)
- net IN1: now also U5.9 (PA4); no longer U5.5 (PA0)
- net IN2: now also U5.10 (PA5); no longer Q2.3 (D), R11.2, U5.6 (PA1)
- net IN3: now also U5.11 (PA6)
- net LED3: now reaches U5.7 (PA2)
- net LED3: now also R19.1
- net IN4: now reaches U5.8 (PA3)
- net IN4: now also Q2.3 (D), R11.2
- net DIP2: no longer names the net of U5.13 (PB0)
- net DIP4: no longer names the net of U5.28 (PB5)
- net TIM3_CH1: no longer names the net of U5.27 (PB4)
- net TIM3_CH2: no longer names the net of U5.26 (PB3)
- new net: JP1.2 (B), R12.1
- new net: D3.2 (A), R18.2
- new net: D2.2 (A), R17.2
- new net: D4.2 (A), R19.2
- new net LED1: R17.1, U5.5 (PA0)
- new net LED2: R18.1, U5.6 (PA1)
- no-connect marks 6 -> 14
Other:
- note added: "LED"
- moved on the sheet: C15, C16, IC1, JP1, R12

Commit message: ビア以外完成
Parts:
- added D10, D5, D6, D7, D8, D9: LED, LED_SMD:LED_0603_1608Metric_Pad1.05x0.95mm_HandSolder, symbol Device:LED
- added R20, R21, R22, R23, R24, R25: 1k, Resistor_SMD:R_0603_1608Metric_Pad0.98x0.95mm_HandSolder, symbol Device:R
Connections:
- net +12V: now also R21.1
- net +3.3V: now also R25.1
- net +5V: now also R24.1
- net +5VP: now also R22.1
- net GNDD: now also D10.1 (K), D5.1 (K), D6.1 (K), D7.1 (K), D8.1 (K), D9.1 (K)
- net IN1: now also U5.10 (PA5); no longer U5.9 (PA4)
- net IN2: now also U5.11 (PA6); no longer U5.10 (PA5)
- net IN3: now also U5.12 (PA7); no longer U5.11 (PA6)
- net IN4: now also U5.9 (PA4); no longer U5.8 (PA3)
- net VCC: now also R20.1
- new net: D9.2 (A), R24.2
- new net: D10.2 (A), R25.2
- new net: D8.2 (A), R23.2
- new net: D7.2 (A), R22.2
- new net: D6.2 (A), R21.2
- new net: D5.2 (A), R20.2
- new net LED4: R23.1, U5.8 (PA3)
- no-connect marks 14 -> 13
Other:
- moved on the sheet: D2, D3, D4, R17, R18, R19

Commit message: 完成
Parts:
- added D11: LED, LED_SMD:LED_0603_1608Metric_Pad1.05x0.95mm_HandSolder, symbol Device:LED
- added R26: 1k, Resistor_SMD:R_0603_1608Metric_Pad0.98x0.95mm_HandSolder, symbol Device:R
Connections:
- net +12VA: now also R26.1
- net GNDD: now also D11.1 (K)
- new net: D11.2 (A), R26.2
Other:
- moved on the sheet: D5, D6, D7, R20, R21, R22
